Commit message: Added params for fingers

File: src/arm/urdf/robot_parameters.xacro (robot description, xacro)
@@ -7,3 +7,5 @@
   <xacro:property name="link_04_name" value="link_04" />
   <xacro:property name="link_05_name" value="link_05" />
+  <xacro:property name="link_06_name" value="finger_01" />
+  <xacro:property name="link_07_name" value="finger_02" />
 </robot>
